Commit message: 再エクスポートしたURDFで木構造の根を胴体に修正
- onshape-to-robot 1.8.3 で再エクスポート（根=Part 1 <6>=胴体、
  11リンク/10ジョイント/全revolute、合計質量10.1058kg）
- リンク名を木構造から機械的に改名（base/lr_*/ll_*）、meshパス整形
- baseフレームをZ軸+90度回転（爪先=+X、上=+Z）
- 左右対称性の検証に基づきLR_HR/LL_HAA/LL_HFE/LR_KFE/LL_FFEの
  軸符号を反転（同符号の関節角で両脚が鏡映対称に動くように）
- limit設定: velocity/effortをモーター定格に基づき設定
  （HR 24/23, HAA 30/15, HFE 30/20, KFE 30/20, FFE 20/23 [Nm/rad/s]）
- 初期姿勢のHAAを0に変更（足裏が水平になるよう）、
  スポーン高さを0.375776mに調整
- 検算・後処理スクリプト一式をtools/に追加
  （verify_export.py, verify_usd.py, postprocess_urdf.py ほか）

Co-Authored-By: Claude Sonnet 5 <noreply@anthropic.com>

File: onshape_export/myrobot_dummy/robot_sim.urdf (robot description, URDF)
Before this commit: robot myrobot_dummy, 11 links, 10 joints
Links:
- link base: mass 1.1195 -> 2.91813
- link ll_ffe: mass 0.604606 -> 0.195902
- link ll_haa: mass 1.0024 -> 0.659153
- link ll_hfe: mass 1.31709 -> 1.09972
- link ll_hr: mass 1.1195 -> 1.02509
- link ll_kfe: mass 0.84373 -> 0.613957
- link lr_ffe: mass 0.604606 -> 0.195902; geometry collision mesh filename=assets/merged/part_1_6_collision.stl; visual mesh filename=assets/merged/part_1_6_visual.stl
- link lr_haa: mass 1.0024 -> 0.659153; geometry collision mesh filename=assets/merged/part_1_3_collision.stl; visual mesh filename=assets/merged/part_1_3_visual.stl
- link lr_hfe: mass 1.31709 -> 1.09972; geometry collision mesh filename=assets/merged/part_1_4_collision.stl; visual mesh filename=assets/merged/part_1_4_visual.stl
- link lr_hr: mass 4.85875 -> 1.02509; geometry collision mesh filename=assets/merged/part_1_2_collision.stl; visual mesh filename=assets/merged/part_1_2_visual.stl
- link lr_kfe: mass 0.843731 -> 0.613958; geometry collision mesh filename=assets/merged/part_1_5_collision.stl; visual mesh filename=assets/merged/part_1_5_visual.stl
Joints:
- joint LL_FFE: axis 0 0 1 -> 0 0 -1; limit lower=-3.141592653589793 upper=3.141592653589793 effort=10 velocity=10 -> lower=-3.141592653589793 upper=3.141592653589793 effort=20 velocity=23
- joint LL_HAA: axis 0 0 1 -> 0 0 -1; limit lower=-3.141592653589793 upper=3.141592653589793 effort=10 velocity=10 -> lower=-3.141592653589793 upper=3.141592653589793 effort=30 velocity=15
- joint LL_HFE: axis 0 0 1 -> 0 0 -1; limit lower=-3.141592653589793 upper=3.141592653589793 effort=10 velocity=10 -> lower=-3.141592653589793 upper=3.141592653589793 effort=30 velocity=20; origin xyz=-0.1125 -0 -0 rpy=-1.5708 0.0318626 -1.5708 -> xyz=-0.1125 -0 0 rpy=-1.5708 0.0318626 -1.5708
- joint LL_HR: limit lower=-3.141592653589793 upper=3.141592653589793 effort=10 velocity=10 -> lower=-3.141592653589793 upper=3.141592653589793 effort=24 velocity=23; origin xyz=0.00160759 0.149991 -0 rpy=3.14159 0 -0.0183197 -> xyz=-0.0886977 0.0544293 0.0761698 rpy=-0.00412115 0.0171439 -3.13765898; parent lr_hr -> base
- joint LL_KFE: limit lower=-3.141592653589793 upper=3.141592653589793 effort=10 velocity=10 -> lower=-3.141592653589793 upper=3.141592653589793 effort=30 velocity=20; origin xyz=0.15 -0 0.0505 rpy=3.14159 -0 -0.212884 -> xyz=0.15 0 0.0505 rpy=3.14159 -0 -0.212884
- joint LR_FFE: limit lower=-3.141592653589793 upper=3.141592653589793 effort=10 velocity=10 -> lower=-3.141592653589793 upper=3.141592653589793 effort=20 velocity=23
- joint LR_HAA: limit lower=-3.141592653589793 upper=3.141592653589793 effort=10 velocity=10 -> lower=-3.141592653589793 upper=3.141592653589793 effort=30 velocity=15; origin xyz=0.0472134 0.0236967 -0.0676576 rpy=-1.58786 -0.00881689 -0.0142351 -> xyz=0 0 -0.075 rpy=-1.5708 -0.00438363 -1.5708; parent base -> lr_hr
- joint LR_HFE: limit lower=-3.141592653589793 upper=3.141592653589793 effort=10 velocity=10 -> lower=-3.141592653589793 upper=3.141592653589793 effort=30 velocity=20
- joint LR_HR: axis 0 0 1 -> 0 0 -1; limit lower=-3.141592653589793 upper=3.141592653589793 effort=10 velocity=10 -> lower=-3.141592653589793 upper=3.141592653589793 effort=24 velocity=23; origin xyz=0.0468992 0.0249812 0.00733077 rpy=3.13716 0.0170655 1.55641 -> xyz=-0.0892368 -0.0955683 0.0755322 rpy=-0.00443454 0.0170655 3.127206327
- joint LR_KFE: axis 0 0 1 -> 0 0 -1; limit lower=-3.141592653589793 upper=3.141592653589793 effort=10 velocity=10 -> lower=-3.141592653589793 upper=3.141592653589793 effort=30 velocity=20
